Commit message: Removed camera drive function, removed single launch file, added end effector xacro and integrated with existing robot xacro

File: ws/src/robot_moveit_config/config/gcr16_2000.urdf.xacro (robot description, xacro)
@@ -7,3 +7,10 @@
     <xacro:include filename="gcr16_2000.ros2_control.xacro" />
     <xacro:gcr16_2000_ros2_control name="FakeSystem" initial_positions_file="$(arg initial_positions_file)"/>
+    <xacro:include filename="$(find robot_moveit_config)/config/end_effector.xacro"/>
+    <joint name="end_effector_joint" type="fixed">
+        <parent link="link_6"/>
+        <child link="bracket_link"/>
+        <!-- Adjust these -->
+        <origin xyz="0 0 0" rpy="0 0 0"/>
+    </joint>
 </robot>

Commit message: Moved arm interface to seperate c++ file, and updated moveit config to attempt to repair TF issue.

File: ws/src/robot_moveit_config/config/gcr16_2000.urdf.xacro (robot description, xacro)
@@ -7,10 +7,5 @@
     <xacro:include filename="gcr16_2000.ros2_control.xacro" />
     <xacro:gcr16_2000_ros2_control name="FakeSystem" initial_positions_file="$(arg initial_positions_file)"/>
-    <xacro:include filename="$(find robot_moveit_config)/config/end_effector.xacro"/>
-    <joint name="end_effector_joint" type="fixed">
-        <parent link="link_6"/>
-        <child link="bracket_link"/>
-        <!-- Adjust these -->
-        <origin xyz="0 0 0" rpy="0 0 0"/>
-    </joint>
+    <xacro:include filename="$(find robot_moveit_config)/models/end_effector.xacro"/>
+    <xacro:bracket_tool parent="link_6"/>
 </robot>
