Commit message: Updated robot model for new dimensions and configured qr_monitor correctly

File: ws/src/robot_model/urdf/gcr16_2000.urdf (robot description, URDF)
Before this commit: robot gcr16_2000, 11 links, 10 joints
Joints:
- joint suction_joint: origin xyz=0 0 0.14605 rpy=0 0 0 -> xyz=0 0 0.2413 rpy=0 0 0
