Commit message: Added dynamic bin support, with control over joints

File: ws/src/robot_model/urdf/bin_filler.urdf (robot description, URDF)
Before this commit: robot bin_filler, 27 links, 26 joints
Links:
- added link base_link
- added link bin_x
- added link bin_y
- added link bin_z
Joints:
- added joint bin_x_joint: type prismatic, parent base_link, child bin_x, axis 1 0 0, limit lower=-5 upper=5 effort=1 velocity=1
- added joint bin_y_joint: type prismatic, parent bin_x, child bin_y, axis 0 1 0, limit lower=-5 upper=5 effort=1 velocity=1
- added joint bin_z_joint: type prismatic, parent bin_y, child bin_z, axis 0 0 1, limit lower=-2 upper=2 effort=1 velocity=1
- added joint dummy_joint: type fixed, parent bin_z, child Top_Frame_2, origin xyz=-0.414 -1.882 0.724 rpy=-0.000 0.000 -1.571

Commit message: Added qr code pose

File: ws/src/robot_model/urdf/bin_filler.urdf (robot description, URDF)
Before this commit: robot bin_filler, 31 links, 30 joints
Links:
- removed link base_link
- removed link bin_x
- removed link bin_y
- removed link bin_z
- added link dummy_link
Joints:
- removed joint bin_x_joint
- removed joint bin_y_joint
- removed joint bin_z_joint
- joint dummy_joint: parent bin_z -> dummy_link

Commit message: Finally got bin scanner working, needed to reconfigure TF tree. It's all good now :)

File: ws/src/robot_model/urdf/bin_filler.urdf (robot description, URDF)
Before this commit: robot bin_filler, 28 links, 27 joints
Joints:
- joint dummy_joint: origin xyz=-0.414 -1.882 0.724 rpy=-0.000 0.000 -1.571 -> xyz=-0.7798 1.882 0.0128 rpy=0.000 0.000 0
