Commit message: Updated bin filler to be simpler URDF

File: ws/src/robot_model/urdf/bin_filler.urdf (robot description, URDF)
Before this commit: robot bin_filler, 28 links, 27 joints
Links:
- removed link 8020-15_Angled_Short_End_Cap_w_QR_Flag_6152026_1
- removed link Angle_Bracket_1
- removed link Angle_Bracket_2
- removed link Angle_Bracket_3
- removed link Angle_Bracket_4
- removed link Apple_Bin_4222026_1
- removed link Apple_Chute_Entrance_4242026_1
- removed link Apple_Chute_Entrance_4242026_2
- removed link Apple_Chute_Entrance_4242026_3
- removed link Apple_Chute_Entrance_4242026_4
- removed link Bottom_Frame_1
- removed link Bottom_Frame_2
- removed link Bottom_Frame_3
- removed link Bottom_Frame_4
- removed link Corner_8020_Series_15_Bracket_4222026_1
- removed link Corner_8020_Series_15_Bracket_4222026_2
- removed link Corner_8020_Series_15_Bracket_4222026_3
- removed link Corner_8020_Series_15_Bracket_4222026_4
- removed link QR_Code_1
- removed link Rubber_Chute_Entrance_Bumper_54206_1
- removed link Rubber_Chute_Entrance_Bumper_54206_2
- removed link Rubber_Chute_Entrance_Bumper_54206_3
- removed link Rubber_Chute_Entrance_Bumper_54206_4
- removed link Top_Frame_1
- removed link Top_Frame_2
- removed link Top_Frame_3
- removed link Top_Frame_4
- added link Bin_Link; collision mesh filename=package://robot_model/meshes/bin_assembly.stl; visual mesh filename=package://robot_model/meshes/bin_assembly.stl
- added link Chute_NE
- added link Chute_NW
- added link Chute_SE
- added link Chute_SW
- added link QR_SE
Joints:
- removed joint Fastened_10
- removed joint Fastened_11
- removed joint Fastened_12
- removed joint Fastened_13
- removed joint Fastened_14
- removed joint Fastened_15
- removed joint Fastened_16
- removed joint Fastened_17
- removed joint Fastened_18
- removed joint Fastened_19
- removed joint Fastened_2
- removed joint Fastened_20
- removed joint Fastened_21
- removed joint Fastened_22
- removed joint Fastened_23
- removed joint Fastened_24
- removed joint Fastened_25
- removed joint Fastened_26
- removed joint Fastened_27
- removed joint Fastened_3
- removed joint Fastened_4
- removed joint Fastened_5
- removed joint Fastened_6
- removed joint Fastened_7
- removed joint Fastened_8
- removed joint Fastened_9
- added joint Chute_NE_Joint: type fixed, parent Bin_Link, child Chute_NE, origin xyz=0.552 0.159 1.107 rpy=0 0 2.356
- added joint Chute_NW_Joint: type fixed, parent Bin_Link, child Chute_NW, origin xyz=-0.159 0.552 1.107 rpy=0 0 -2.356
- added joint Chute_SE_Joint: type fixed, parent Bin_Link, child Chute_SE, origin xyz=0.159 -0.552 1.107 rpy=0 0 0.785
- added joint Chute_SW_Joint: type fixed, parent Bin_Link, child Chute_SW, origin xyz=-0.552 -0.159 1.107 rpy=0 0 -0.785
- added joint QR_SE_Joint: type fixed, parent Bin_Link, child QR_SE, origin xyz=0.302 -0.302 1.129 rpy=0.785 0.000 0.785
- joint dummy_joint: child Top_Frame_2 -> Bin_Link; origin xyz=-0.7798 1.882 0.0128 rpy=0.000 0.000 0 -> xyz=-0.5969 0.5969 0.0 rpy=0.0 0.0 0.0

Commit message: Initial commit for scout_camera_scanner

File: ws/src/robot_model/urdf/bin_filler.urdf (robot description, URDF)
Before this commit: robot bin_filler, 7 links, 6 joints
Links:
- added link scout_link; visual mesh filename=package://robot_model/meshes/DS87-Mechanical_Outline_3D.STP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 scale=0.002 0.002 0.002
Joints:
- added joint Scout_Cam_Static: type fixed, parent Bin_Link, child scout_link, origin xyz=-0.5969 1.2038 0.762 rpy=-1.57079633 -1.57079633 0.0

Commit message: Adding pick and place pipeline test along with compatibility and bugfixes. Begin work on scan pose system

File: ws/src/robot_model/urdf/bin_filler.urdf (robot description, URDF)
Before this commit: robot bin_filler, 8 links, 7 joints
Joints:
- joint Scout_Cam_Static: origin xyz=-0.5969 1.2038 0.762 rpy=-1.57079633 -1.57079633 0.0 -> xyz=-0.5969 1.2192 0.762 rpy=-1.57079633 -1.57079633 0.0

File: ws/src/robot_model/urdf/gcr16_2000.urdf (robot description, URDF)
Before this commit: robot gcr16_2000, 11 links, 10 joints
Links:
- link bracket_link: geometry collision box size=0.1778 0.3048 0.2032; visual mesh filename=package://robot_model/meshes/End_Effector_Bracket_4.2.2026.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 scale=0.001 0.001 0.001
- link camera_link: geometry visual mesh filename=package://robot_model/meshes/DS87-Mechanical_Outline_3D.STP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 scale=0.002 0.002 0.002

File: ws/src/robot_model/urdf/robot_workspace.urdf (robot description, URDF)
Before this commit: robot workspace, 4 links, 3 joints
Links:
- link arm_1_main_workspace: geometry visual box size=0.1 0.609 1.2192
